File: elektronics/eye/Eye.kicad_pcb (KiCad board)
At the start: 2 copper layers, 30.5 x 16.5 mm, 4 parts, among them CON1 PI, CON2 HC-SR04

Commit message: first little remote control by client / new podest design / pcb with drill holes
Parts:
- moved CON2 6.38 mm to (51.4, 40.6)
- moved R1 6.38 mm to (42.5, 29.2)
- moved R2 6.38 mm to (37.5, 29.2)
- moved CON1 6.38 mm to (31.1, 38.1)
Other:
- board size 30.5 x 16.5 mm -> 30 x 26 mm
Changed lines of the file:
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@@
   (general
     (thickness 1.6)
-    (drawings 4)
+    (drawings 7)
     (tracks 19)
     (zones 0)
@@
     (pad_drill 0.762)
     (pad_to_mask_clearance 0)
-    (aux_axis_origin 0 0)
+    (aux_axis_origin 77 36)
     (visible_elements FFFFFF7F)
     (pcbplotparams
@@
   )
   (module Connector_JAE:JAE_LY20-4P-DT1_2x02_P2.00mm_Vertical (layer F.Cu)
-    (at 30.48 31.75 180)
+    (at 31.115 38.1 180)
     (descr "Molex LY 20 series connector, LY20-4P-DT1, 2 Circuits (http://www.jae.com/z-en/pdf_download_exec.cfm?param=SJ103130.pdf), generated with kicad-footprint-generator")
     (tags "connector JAE  side entry")
@@
   )
   (module Connector_JAE:JAE_LY20-10P-DT1_2x05_P2.00mm_Vertical (layer F.Cu)
-    (at 50.8 34.29 180)
+    (at 51.435 40.64 180)
     (descr "Molex LY 20 series connector, LY20-10P-DT1, 5 Circuits (http://www.jae.com/z-en/pdf_download_exec.cfm?param=SJ103130.pdf), generated with kicad-footprint-generator")
     (tags "connector JAE  side entry")
@@
   )
   (module Resistor_THT:R_Axial_DIN0207_L6.3mm_D2.5mm_P10.16mm_Horizontal (layer F.Cu)
-    (at 41.91 22.86 270)
+    (at 42.545 29.21 270)
     (descr "Resistor, Axial_DIN0207 series, Axial, Horizontal, pin pitch=10.16mm, 0.25W = 1/4W, length*diameter=6.3*2.5mm^2, http://cdn-reichelt.de/documents/datenblatt/B400/1_4W%23YAG.pdf")
     (tags "Resistor Axial_DIN0207 series Axial Horizontal pin pitch 10.16mm 0.25W = 1/4W length 6.3mm diameter 2.5mm")
@@
   )
   (module Resistor_THT:R_Axial_DIN0207_L6.3mm_D2.5mm_P10.16mm_Horizontal (layer F.Cu)
-    (at 36.83 22.86 270)
+    (at 37.465 29.21 270)
     (descr "Resistor, Axial_DIN0207 series, Axial, Horizontal, pin pitch=10.16mm, 0.25W = 1/4W, length*diameter=6.3*2.5mm^2, http://cdn-reichelt.de/documents/datenblatt/B400/1_4W%23YAG.pdf")
     (tags "Resistor Axial_DIN0207 series Axial Horizontal pin pitch 10.16mm 0.25W = 1/4W length 6.3mm diameter 2.5mm")
@@
     )
   )
-  (gr_line (start 54.61 21.59) (end 24.13 21.59) (layer Edge.Cuts) (width 0.1))
-  (gr_line (start 54.61 38.1) (end 54.61 21.59) (layer Edge.Cuts) (width 0.1))
-  (gr_line (start 24.13 38.1) (end 54.61 38.1) (layer Edge.Cuts) (width 0.1))
-  (gr_line (start 24.13 21.59) (end 24.13 38.1) (layer Edge.Cuts) (width 0.1))
-  (segment (start 48.200001 32.889999) (end 45.850001 32.889999) (width 0.25) (layer F.Cu) (net 1))
-  (segment (start 48.8 32.29) (end 48.200001 32.889999) (width 0.25) (layer F.Cu) (net 1))
-  (segment (start 45.850001 32.889999) (end 43.18 35.56) (width 0.25) (layer F.Cu) (net 1))
-  (segment (start 30.48 32.35) (end 30.48 31.75) (width 0.25) (layer F.Cu) (net 1))
-  (segment (start 33.69 35.56) (end 30.48 32.35) (width 0.25) (layer F.Cu) (net 1))
-  (segment (start 43.18 35.56) (end 33.69 35.56) (width 0.25) (layer F.Cu) (net 1))
-  (segment (start 41.56 28.29) (end 36.83 33.02) (width 0.25) (layer F.Cu) (net 2))
-  (segment (start 48.8 28.29) (end 41.56 28.29) (width 0.25) (layer F.Cu) (net 2))
-  (segment (start 33.75 33.02) (end 30.48 29.75) (width 0.25) (layer F.Cu) (net 2))
-  (segment (start 36.83 33.02) (end 33.75 33.02) (width 0.25) (layer F.Cu) (net 2))
-  (segment (start 48.8 34.29) (end 46.99 34.29) (width 0.25) (layer F.Cu) (net 3))
-  (segment (start 46.99 34.29) (end 44.45 36.83) (width 0.25) (layer F.Cu) (net 3))
-  (segment (start 33.56 36.83) (end 28.48 31.75) (width 0.25) (layer F.Cu) (net 3))
-  (segment (start 44.45 36.83) (end 33.56 36.83) (width 0.25) (layer F.Cu) (net 3))
-  (segment (start 41.91 22.86) (end 36.83 22.86) (width 0.25) (layer F.Cu) (net 4))
-  (segment (start 35.37 22.86) (end 28.48 29.75) (width 0.25) (layer F.Cu) (net 4))
-  (segment (start 36.83 22.86) (end 35.37 22.86) (width 0.25) (layer F.Cu) (net 4))
-  (segment (start 44.64 30.29) (end 41.91 33.02) (width 0.25) (layer F.Cu) (net 10))
-  (segment (start 48.8 30.29) (end 44.64 30.29) (width 0.25) (layer F.Cu) (net 10))
+  (target plus (at 40 46) (size 3) (width 0.1) (layer Edge.Cuts))
+  (target plus (at 40 26) (size 3) (width 0.1) (layer Edge.Cuts))
+  (dimension 20 (width 0.15) (layer F.SilkS)
+    (gr_text "20,000 mm" (at 14.7 36 270) (layer F.SilkS)
+      (effects (font (size 1 1) (thickness 0.15)))
+    )
+    (feature1 (pts (xy 21 46) (xy 15.413579 46)))
+    (feature2 (pts (xy 21 26) (xy 15.413579 26)))
+    (crossbar (pts (xy 16 26) (xy 16 46)))
+    (arrow1a (pts (xy 16 46) (xy 15.413579 44.873496)))
+    (arrow1b (pts (xy 16 46) (xy 16.586421 44.873496)))
+    (arrow2a (pts (xy 16 26) (xy 15.413579 27.126504)))
+    (arrow2b (pts (xy 16 26) (xy 16.586421 27.126504)))
+  )
+  (gr_line (start 55 23) (end 25 23) (layer Edge.Cuts) (width 0.1))
+  (gr_line (start 55 49) (end 55 23) (layer Edge.Cuts) (width 0.1))
+  (gr_line (start 25 49) (end 55 49) (layer Edge.Cuts) (width 0.1))
+  (gr_line (start 25 23) (end 25 49) (layer Edge.Cuts) (width 0.1))
+  (segment (start 48.835001 39.239999) (end 46.485001 39.239999) (width 0.25) (layer F.Cu) (net 1))
+  (segment (start 49.435 38.64) (end 48.835001 39.239999) (width 0.25) (layer F.Cu) (net 1))
+  (segment (start 46.485001 39.239999) (end 43.815 41.91) (width 0.25) (layer F.Cu) (net 1))
+  (segment (start 31.115 38.7) (end 31.115 38.1) (width 0.25) (layer F.Cu) (net 1))
+  (segment (start 34.325 41.91) (end 31.115 38.7) (width 0.25) (layer F.Cu) (net 1))
+  (segment (start 43.815 41.91) (end 34.325 41.91) (width 0.25) (layer F.Cu) (net 1))
+  (segment (start 42.195 34.64) (end 37.465 39.37) (width 0.25) (layer F.Cu) (net 2))
+  (segment (start 49.435 34.64) (end 42.195 34.64) (width 0.25) (layer F.Cu) (net 2))
+  (segment (start 34.385 39.37) (end 31.115 36.1) (width 0.25) (layer F.Cu) (net 2))
+  (segment (start 37.465 39.37) (end 34.385 39.37) (width 0.25) (layer F.Cu) (net 2))
+  (segment (start 49.435 40.64) (end 47.625 40.64) (width 0.25) (layer F.Cu) (net 3))
+  (segment (start 47.625 40.64) (end 45.085 43.18) (width 0.25) (layer F.Cu) (net 3))
+  (segment (start 34.195 43.18) (end 29.115 38.1) (width 0.25) (layer F.Cu) (net 3))
+  (segment (start 45.085 43.18) (end 34.195 43.18) (width 0.25) (layer F.Cu) (net 3))
+  (segment (start 42.545 29.21) (end 37.465 29.21) (width 0.25) (layer F.Cu) (net 4))
+  (segment (start 36.005 29.21) (end 29.115 36.1) (width 0.25) (layer F.Cu) (net 4))
+  (segment (start 37.465 29.21) (end 36.005 29.21) (width 0.25) (layer F.Cu) (net 4))
+  (segment (start 45.275 36.64) (end 42.545 39.37) (width 0.25) (layer F.Cu) (net 10))
+  (segment (start 49.435 36.64) (end 45.275 36.64) (width 0.25) (layer F.Cu) (net 10))
 )
